Commit message: update deploy

File: b2/wbc_deploy/reference_scripts/b2z1.urdf (robot description, URDF)
Before this commit: robot b2z1_description, 47 links, 46 joints
Links:
- link FL_thigh: geometry collision box size=0.25 0.028 0.04; visual mesh filename=../meshes/FL_thigh.dae
- link link00: mass 0.47247481+0.66000 -> 1.3247481
Joints:
- joint FL_calf_joint: limit lower=-2.82 upper=-0.43 effort=320 velocity=14 -> lower=-2.82 upper=-1.0 effort=320 velocity=14
- joint FL_hip_joint: limit lower=-0.87 upper=0.87 effort=200 velocity=23 -> lower=-0.2 upper=0.2 effort=200 velocity=23
- joint FL_thigh_joint: limit lower=-0.94 upper=4.69 effort=200 velocity=23 -> lower=-0.94 upper=1.0 effort=200 velocity=23
- joint FR_calf_joint: limit lower=-2.82 upper=-0.43 effort=320 velocity=14 -> lower=-2.82 upper=-1.0 effort=320 velocity=14
- joint FR_hip_joint: limit lower=-0.87 upper=0.87 effort=200 velocity=23 -> lower=-0.2 upper=0.2 effort=200 velocity=23
- joint FR_thigh_joint: limit lower=-0.94 upper=4.69 effort=200 velocity=23 -> lower=-0.94 upper=1.0 effort=200 velocity=23
- joint RL_calf_joint: limit lower=-2.82 upper=-0.43 effort=320 velocity=14 -> lower=-2.82 upper=-1.0 effort=320 velocity=14
- joint RL_hip_joint: limit lower=-0.87 upper=0.87 effort=200 velocity=23 -> lower=-0.2 upper=0.2 effort=200 velocity=23
- joint RL_thigh_joint: limit lower=-0.94 upper=4.69 effort=200 velocity=23 -> lower=-0.94 upper=1.0 effort=200 velocity=23
- joint RR_calf_joint: limit lower=-2.82 upper=-0.43 effort=320 velocity=14 -> lower=-2.82 upper=-1.0 effort=320 velocity=14
- joint RR_hip_joint: limit lower=-0.87 upper=0.87 effort=200 velocity=23 -> lower=-0.2 upper=0.2 effort=200 velocity=23
- joint RR_thigh_joint: limit lower=-0.94 upper=4.69 effort=200 velocity=23 -> lower=-0.94 upper=1.0 effort=200 velocity=23
- joint z1_elbow: limit lower=-4.782202150464463 upper=0.0 effort=30.0 velocity=10 -> lower=-3.0 upper=0.0 effort=30.0 velocity=10
- joint z1_shoulder: limit lower=0.0 upper=3.141592653589793 effort=60.0 velocity=10 -> lower=0.0 upper=2.8 effort=60.0 velocity=10
